File: PCB/SR_redesign/SR_digit_board/SR_digit_board.kicad_sch (KiCad schematic)
At the start: 82 parts, among them J1 Conn_02x07_Counter_Clockwise, J2 Conn_01x09, J3 Conn_01x10, J4 Conn_01x09, Q1 MPSA92-AP, Q10 MPSA42-AP, Q11 MPSA42-AP, Q12 MPSA42-AP, Q2 MPSA92-AP, Q3 MPSA92-AP, Q4 MPSA42-AP, Q5 MPSA42-AP, Q6 MPSA42-AP, Q7 MPSA92-AP, Q8 MPSA92-AP, Q9 MPSA92-AP, U1 74141, U2 74141, U3 74141, U4 SN74HC595N, U5 SN74HC595N, U6 SN74HC595N, U7 ATMEGA328PB-AU

Commit message: SR redesign - added buttons. copypasted seconds
Parts:
- removed TP1, TP10, TP11, TP12, TP13, TP14, TP15, TP16, TP17, TP18, TP19, TP2, TP20, TP21, TP22, TP23, TP24, TP3, TP4, TP5, TP6, TP7, TP8, TP9: RCU-0C, digikey-footprints:PROBE_PAD_0603, symbol dk_Test-Points:RCU-0C
- added SW1, SW2, SW3: SW_Push_SPDT, symbol Switch:SW_Push_SPDT
Connections:
- net GND: now also SW1.3 (C), SW2.3 (C), SW3.3 (C)
- net Switch0: now reaches U7.23 (PC0)
- net Switch0: now also SW1.2 (B)
- net Switch1: now reaches U7.24 (PC1)
- net Switch1: now also SW2.2 (B)
- net Switch2: now reaches U7.25 (PC2)
- net Switch2: now also SW3.2 (B)
- no-connect marks 36 -> 33

Commit message: SR redesign - added atmega support components, still need xtal footprint
Parts:
- added C1, C2: 22p, Capacitor_SMD:C_0805_2012Metric_Pad1.18x1.45mm_HandSolder, symbol Device:C
- added R25: 15k, Resistor_SMD:R_0805_2012Metric_Pad1.20x1.40mm_HandSolder, symbol Device:R_US
- added Y1: 16MHz, symbol Device:Crystal
- SW1, SW2, SW3: footprint (none) -> Connector_PinHeader_2.54mm:PinHeader_1x02_P2.54mm_Vertical
Connections:
- net GND: now also C1.1, C2.1, R25.2
- net at D10.1 (K), D8.1 (K), U7.4 (VCC): now also U7.18 (AVCC)
- net at U7.13 (PB1): now also C2.2, Y1.1
- net at U7.14 (PB2): now also C1.2, Y1.2
- net at U7.29 (PC6): now also R25.1
- no-connect marks 33 -> 29

Commit message: SR redesign - most of the layout seems to be there. need a power supply
Parts:
- removed D7, D9: 1N4001, Diode_THT:D_DO-41_SOD81_P10.16mm_Horizontal, symbol Diode:1N4001
- Y1: footprint (none) -> Crystal:Crystal_HC18-U_Vertical
Connections:
- net GND: now also SW1.1 (A), SW2.1 (A), SW3.1 (A)
- net ORpower: now reaches J1.6 (Pin_6)
- net ORpower: now also D10.1 (K), D8.1 (K), U7.18 (AVCC), U7.4 (VCC)
- net at C2.2, U7.13 (PB1): now also Y1.2; no longer Y1.1
- net at C1.2, U7.14 (PB2): now also Y1.1; no longer Y1.2
Other:
- moved on the sheet: Y1
Changed lines of the file:
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@@
   (junction (at 180.34 148.59) (diameter 0) (color 0 0 0 0)
   )
+  (junction (at 280.67 62.23) (diameter 0) (color 0 0 0 0)
+  )
   (junction (at 83.82 97.79) (diameter 0) (color 0 0 0 0)
   )
@@
   (junction (at 91.44 152.4) (diameter 0) (color 0 0 0 0)
   )
+  (junction (at 280.67 74.93) (diameter 0) (color 0 0 0 0)
+  )
   (junction (at 53.34 99.06) (diameter 0) (color 0 0 0 0)
   )
@@
   (junction (at 185.42 95.25) (diameter 0) (color 0 0 0 0)
   )
+  (junction (at 280.67 80.01) (diameter 0) (color 0 0 0 0)
+  )
   (junction (at 93.98 92.71) (diameter 0) (color 0 0 0 0)
   )
@@
   (junction (at 106.68 29.21) (diameter 0) (color 0 0 0 0)
   )
+  (junction (at 280.67 44.45) (diameter 0) (color 0 0 0 0)
+  )
   (junction (at 205.74 46.99) (diameter 0) (color 0 0 0 0)
   )
@@
   (junction (at 185.42 153.67) (diameter 0) (color 0 0 0 0)
   )
-  (junction (at 217.17 124.46) (diameter 0) (color 0 0 0 0)
-  )
   (junction (at 267.97 115.57) (diameter 0) (color 0 0 0 0)
   )
@@
     (stroke (width 0) (type default) (color 0 0 0 0))
   )
+  (wire (pts (xy 280.67 57.15) (xy 280.67 62.23))
+    (stroke (width 0) (type default) (color 0 0 0 0))
+  )
   (wire (pts (xy 212.09 90.17) (xy 227.33 90.17))
     (stroke (width 0) (type default) (color 0 0 0 0))
@@
     (stroke (width 0) (type default) (color 0 0 0 0))
   )
+  (wire (pts (xy 280.67 73.66) (xy 280.67 74.93))
+    (stroke (width 0) (type default) (color 0 0 0 0))
+  )
   (wire (pts (xy 118.11 154.94) (xy 86.36 154.94))
     (stroke (width 0) (type default) (color 0 0 0 0))
@@
     (stroke (width 0) (type default) (color 0 0 0 0))
   )
-  (wire (pts (xy 217.17 124.46) (xy 215.9 124.46))
-    (stroke (width 0) (type default) (color 0 0 0 0))
-  )
   (wire (pts (xy 115.57 34.29) (xy 96.52 34.29))
     (stroke (width 0) (type default) (color 0 0 0 0))
@@
     (stroke (width 0) (type default) (color 0 0 0 0))
   )
-  (wire (pts (xy 208.28 120.65) (xy 208.28 124.46))
-    (stroke (width 0) (type default) (color 0 0 0 0))
-  )
   (wire (pts (xy 93.98 151.13) (xy 93.98 157.48))
     (stroke (width 0) (type default) (color 0 0 0 0))
@@
     (stroke (width 0) (type default) (color 0 0 0 0))
   )
+  (wire (pts (xy 280.67 74.93) (xy 280.67 80.01))
+    (stroke (width 0) (type default) (color 0 0 0 0))
+  )
   (wire (pts (xy 219.71 114.3) (xy 217.17 114.3))
     (stroke (width 0) (type default) (color 0 0 0 0))
@@
     (stroke (width 0) (type default) (color 0 0 0 0))
   )
+  (wire (pts (xy 280.67 39.37) (xy 280.67 44.45))
+    (stroke (width 0) (type default) (color 0 0 0 0))
+  )
   (wire (pts (xy 199.39 78.74) (xy 199.39 85.09))
     (stroke (width 0) (type default) (color 0 0 0 0))
@@
     (stroke (width 0) (type default) (color 0 0 0 0))
   )
-  (wire (pts (xy 217.17 114.3) (xy 217.17 124.46))
-    (stroke (width 0) (type default) (color 0 0 0 0))
-  )
-  (wire (pts (xy 218.44 124.46) (xy 217.17 124.46))
-    (stroke (width 0) (type default) (color 0 0 0 0))
-  )
   (wire (pts (xy 243.84 144.78) (xy 256.54 144.78))
     (stroke (width 0) (type default) (color 0 0 0 0))
@@
     )
   )
+  (global_label "ORpower" (shape input) (at 227.33 30.48 90) (fields_autoplaced)
+    (effects (font (size 1.27 1.27)) (justify left))
+    (property "Intersheet References" "${INTERSHEET_REFS}" (id 0) (at 227.2506 19.9631 90)
+      (effects (font (size 1.27 1.27)) (justify left) hide)
+    )
+  )
   (global_label "h_LO" (shape input) (at 21.59 67.31 180) (fields_autoplaced)
     (effects (font (size 1.27 1.27)) (justify right))
@@
     )
   )
-  (global_label "Vbatt" (shape input) (at 226.06 124.46 0) (fields_autoplaced)
-    (effects (font (size 1.27 1.27)) (justify left))
-    (property "Intersheet References" "${INTERSHEET_REFS}" (id 0) (at 233.3112 124.3806 0)
-      (effects (font (size 1.27 1.27)) (justify left) hide)
-    )
-  )
   (global_label "Switch2" (shape input) (at 270.51 77.47 180) (fields_autoplaced)
     (effects (font (size 1.27 1.27)) (justify right))
@@
     )
   )
+  (global_label "ORpower" (shape input) (at 217.17 114.3 180) (fields_autoplaced)
+    (effects (font (size 1.27 1.27)) (justify right))
+    (property "Intersheet References" "${INTERSHEET_REFS}" (id 0) (at 206.6531 114.3794 0)
+      (effects (font (size 1.27 1.27)) (justify right) hide)
+    )
+  )
   (global_label "m_HI" (shape input) (at 44.45 111.76 180) (fields_autoplaced)
     (effects (font (size 1.27 1.27)) (justify right))
@@
     (pin "3")
   )
-  (symbol (lib_id "power:+5V") (at 208.28 120.65 0) (unit 1)
-    (in_bom yes) (on_board yes)
-    (property "Reference" "#PWR013" (id 0) (at 208.28 124.46 0)
-      (effects (font (size 1.27 1.27)) hide)
-    )
-    (property "Value" "+5V" (id 1) (at 208.28 115.57 0))
-    (property "Footprint" "" (id 2) (at 208.28 120.65 0)
-      (effects (font (size 1.27 1.27)) hide)
-    )
-    (property "Datasheet" "" (id 3) (at 208.28 120.65 0)
-      (effects (font (size 1.27 1.27)) hide)
-    )
-    (pin "1")
-  )
-  (symbol (lib_id "Diode:1N4001") (at 222.25 124.46 0) (unit 1)
-    (in_bom yes) (on_board yes) (fields_autoplaced)
-    (property "Reference" "D9" (id 0) (at 222.25 118.11 0))
-    (property "Value" "1N4001" (id 1) (at 222.25 120.65 0))
-    (property "Footprint" "Diode_THT:D_DO-41_SOD81_P10.16mm_Horizontal" (id 2) (at 222.25 128.905 0)
-      (effects (font (size 1.27 1.27)) hide)
-    )
-    (property "Datasheet" "http://www.vishay.com/docs/88503/1n4001.pdf" (id 3) (at 222.25 124.46 0)
-      (effects (font (size 1.27 1.27)) hide)
-    )
-    (pin "1")
-    (pin "2")
-  )
   (symbol (lib_id "Device:R_US") (at 41.91 124.46 90) (unit 1)
     (in_bom yes) (on_board yes) (fields_autoplaced)
@@
     (pin "2")
   )
-  (symbol (lib_id "Device:Crystal") (at 209.55 44.45 180) (unit 1)
+  (symbol (lib_id "Device:Crystal") (at 209.55 44.45 0) (mirror x) (unit 1)
     (in_bom yes) (on_board yes) (fields_autoplaced)
     (property "Reference" "Y1" (id 0) (at 209.55 36.83 0))
     (property "Value" "16MHz" (id 1) (at 209.55 39.37 0))
-    (property "Footprint" "" (id 2) (at 209.55 44.45 0)
+    (property "Footprint" "Crystal:Crystal_HC18-U_Vertical" (id 2) (at 209.55 44.45 0)
       (effects (font (size 1.27 1.27)) hide)
     )
@@
     (pin "A")
   )
-  (symbol (lib_id "Diode:1N4001") (at 212.09 124.46 180) (unit 1)
-    (in_bom yes) (on_board yes) (fields_autoplaced)
-    (property "Reference" "D7" (id 0) (at 212.09 118.11 0))
-    (property "Value" "1N4001" (id 1) (at 212.09 120.65 0))
-    (property "Footprint" "Diode_THT:D_DO-41_SOD81_P10.16mm_Horizontal" (id 2) (at 212.09 120.015 0)
-      (effects (font (size 1.27 1.27)) hide)
-    )
-    (property "Datasheet" "http://www.vishay.com/docs/88503/1n4001.pdf" (id 3) (at 212.09 124.46 0)
-      (effects (font (size 1.27 1.27)) hide)
-    )
-    (pin "1")
-    (pin "2")
-  )
   (symbol (lib_id "Switch:SW_Push_SPDT") (at 275.59 59.69 0) (unit 1)
     (in_bom yes) (on_board yes) (fields_autoplaced)
@@
       (reference "#PWR012") (unit 1) (value "GND") (footprint "")
     )
-    (path "/154eb887-76aa-4f51-a220-6a07b4459118"
-      (reference "#PWR013") (unit 1) (value "+5V") (footprint "")
-    )
     (path "/55034d7f-c64b-4d73-b96a-f53186671462"
       (reference "#PWR014") (unit 1) (value "+5V") (footprint "")
@@
       (reference "D6") (unit 1) (value "IN-12") (footprint "nixies-us:nixies-us-IN-12-DSUB")
     )
-    (path "/c129440e-af99-48a6-bfa5-df35ae4d1651"
-      (reference "D7") (unit 1) (value "1N4001") (footprint "Diode_THT:D_DO-41_SOD81_P10.16mm_Horizontal")
-    )
     (path "/5154868c-b118-4f0a-997e-3b02b6308771"
       (reference "D8") (unit 1) (value "1N4001") (footprint "Diode_THT:D_DO-41_SOD81_P10.16mm_Horizontal")
     )
-    (path "/17bcfca6-84d3-4088-90a7-1f76dd253ae6"
-      (reference "D9") (unit 1) (value "1N4001") (footprint "Diode_THT:D_DO-41_SOD81_P10.16mm_Horizontal")
-    )
     (path "/aea9c950-b0ce-4d0a-bbf5-552c0324a04e"
       (reference "D10") (unit 1) (value "1N4001") (footprint "Diode_THT:D_DO-41_SOD81_P10.16mm_Horizontal")
@@
     )
     (path "/a1a6d320-8a24-4c6a-ba7b-e992540fc3e3"
-      (reference "Y1") (unit 1) (value "16MHz") (footprint "")
+      (reference "Y1") (unit 1) (value "16MHz") (footprint "Crystal:Crystal_HC18-U_Vertical")
     )
   )
