File: PCB/SR_redesign/SR_digit_board/SR_digit_board.kicad_pcb (KiCad board)
At the start: 2 copper layers, 234.1 x 84 mm, 64 parts, among them J1 Conn_02x07_Counter_Clockwise, J2 Conn_01x09, J3 Conn_01x10, J4 Conn_01x09, Q1 MPSA92-AP, Q10 MPSA42-AP, Q11 MPSA42-AP, Q12 MPSA42-AP, Q2 MPSA92-AP, Q3 MPSA92-AP, Q4 MPSA42-AP, Q5 MPSA42-AP, Q6 MPSA42-AP, Q7 MPSA92-AP, Q8 MPSA92-AP, Q9 MPSA92-AP, SW1 SW_Push_SPDT, SW2 SW_Push_SPDT, SW3 SW_Push_SPDT, U1 74141, U2 74141, U3 74141, U4 SN74HC595N, U5 SN74HC595N, U6 SN74HC595N, U7 ATMEGA328PB-AU, Y1 16MHz

Commit message: SR redesign - possible complete board with gerbers. included power supply on boards. traces bridge regions. might need to revisit if the ribbon cable spacing is different or if we want to nudge the tube pairs closer to each other
Parts:
- removed the J4 at (176.1, 113.7)
- added 100uH: 100u, Inductor_THT:L_Radial_D8.7mm_P5.00mm_Fastron_07HCP, B.Cu at (120.0, 155.0)
- added 10k: 10k, Resistor_THT:R_Axial_DIN0207_L6.3mm_D2.5mm_P7.62mm_Horizontal, B.Cu at (147.0, 149.3)
- added 1k: 1k, Resistor_THT:R_Axial_DIN0207_L6.3mm_D2.5mm_P7.62mm_Horizontal, B.Cu at (139.4, 146.1)
- added 1k Pot: 1k, Potentiometer_THT:Potentiometer_Bourns_3386P_Vertical, B.Cu at (109.6, 156.2)
- added 1k: 1k, Resistor_THT:R_Axial_DIN0207_L6.3mm_D2.5mm_P7.62mm_Horizontal, B.Cu at (126.2, 153.0)
- added 1k: 1k, Resistor_THT:R_Axial_DIN0207_L6.3mm_D2.5mm_P7.62mm_Horizontal, B.Cu at (87.9, 137.9)
- added 1u: 1u, Capacitor_THT:CP_Radial_D6.3mm_P2.50mm, B.Cu at (96.1, 135.7)
- added 2.2n: 2.2n, Capacitor_THT:C_Disc_D12.5mm_W5.0mm_P10.00mm, B.Cu at (136.8, 159.1)
- added 220k: 220k, Resistor_THT:R_Axial_DIN0207_L6.3mm_D2.5mm_P7.62mm_Horizontal, B.Cu at (100.0, 151.3)
- added 220nTANT: 220nTANT, Capacitor_THT:C_Disc_D3.8mm_W2.6mm_P2.50mm, B.Cu at (161.2, 153.6)
- added 220nTANT: 220nTANT, Capacitor_THT:C_Disc_D3.8mm_W2.6mm_P2.50mm, B.Cu at (161.2, 158.4)
- added 33k: 33k, Resistor_THT:R_Axial_DIN0207_L6.3mm_D2.5mm_P7.62mm_Horizontal, B.Cu at (123.5, 151.1)
- added 4.7k: 4.7k, Resistor_THT:R_Axial_DIN0207_L6.3mm_D2.5mm_P7.62mm_Horizontal, B.Cu at (100.0, 133.8)
- added 470: 470, Resistor_THT:R_Axial_DIN0207_L6.3mm_D2.5mm_P7.62mm_Horizontal, B.Cu at (106.7, 146.6)
- added 470u: 470u, Capacitor_THT:CP_Radial_D10.0mm_P5.00mm, B.Cu at (173.6, 153.9)
- added 47p: 47p, Capacitor_THT:C_Disc_D3.4mm_W2.1mm_P2.50mm, B.Cu at (84.9, 130.3)
- added <-D: D, Diode_THT:D_DO-41_SOD81_P2.54mm_Vertical_KathodeUp, B.Cu at (157.8, 146.9)
- added BC547: BC547, Package_TO_SOT_THT:TO-92_Inline_Wide, B.Cu at (122.8, 147.2)
- added BarrelJack: Barrel_Jack, Connector_PinHeader_2.54mm:PinHeader_1x02_P2.54mm_Vertical, B.Cu at (161.2, 149.5)
- added D11: D, Diode_THT:D_DO-41_SOD81_P7.62mm_Horizontal, B.Cu at (98.5, 130.2)
- added D9: D_ALT, Diode_THT:D_DO-35_SOD27_P7.62mm_Horizontal, B.Cu at (96.3, 140.6)
- added F1: Polyfuse, Fuse:Fuse_Bourns_MF-RG300, B.Cu at (154.8, 147.2)
- added IRF740: IRF740, Package_TO_SOT_THT:TO-220-3_Horizontal_TabUp, B.Cu at (91.7, 140.6)
- added J7: Conn_01x09, Connector_PinHeader_2.54mm:PinHeader_2x05_P2.54mm_Vertical, F.Cu at (176.1, 107.2)
- added MC7805 Reg: MC7805CT-BP, Package_TO_SOT_THT:TO-220-3_Horizontal_TabUp, B.Cu at (158.3, 159.2)
- added MPSA55: MPSA55-AP, digikey-footprints:TO-92-3_Formed_Leads, B.Cu at (98.9, 154.5)
- added NE555: NE555P, digikey-footprints:DIP-8_W7.62mm, B.Cu at (136.9, 152.9)
- 595 SR: renamed from U5
- 595 SR: renamed from U4
- 595 SR: renamed from U6
- 8025 RTC: renamed from J1
- BAT1, D10, D8, SW1, SW2, SW3: moved to B.Cu
- moved BAT1 16.6 mm to (177.4, 129.6)
- moved 16Mhz 6.41 mm to (217.1, 147.9)
- moved 22p 6.41 mm to (226.8, 148.9)
- moved 22p 6.41 mm to (212.4, 148.9)
- moved MPSA42 6.41 mm to (60.5, 128.9)
- moved MPSA42 6.41 mm to (145.4, 128.9)
- moved MPSA42 6.41 mm to (230.4, 128.9)
- moved 15k 6.41 mm to (209.8, 123.4)
- moved 15k 6.41 mm to (124.8, 123.4)
- moved 15k 6.41 mm to (68.7, 123.4)
- moved 15k 6.41 mm to (238.7, 123.4)
- moved 15k 6.41 mm to (39.8, 123.4)
- moved 15k 6.41 mm to (153.7, 123.4)
- moved 33k 6.41 mm to (44.8, 127.4)
- moved 33k 6.41 mm to (54.8, 126.0)
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- renumbered R6 to 100k, R16 to 100k, R20 to 100k, R8 to 100k, R18 to 100k, R4 to 100k, R15 to 15k, R14 to 15k, R1 to 15k, R3 to 15k, R13 to 15k, R2 to 15k, Y1 to 16Mhz, C2 to 22p, C1 to 22p, U7 to 328P, R22 to 33k, R10 to 33k, R12 to 33k, R24 to 33k, R11 to 33k, R23 to 33k, R17 to 470k, R21 to 470k, R9 to 470k, R19 to 470k, R5 to 470k, R7 to 470k, U1 to K155ID1, U3 to K155ID1, U2 to K155ID1, Q4 to MPSA42, Q5 to MPSA42, Q12 to MPSA42, Q6 to MPSA42, Q11 to MPSA42, Q10 to MPSA42, Q9 to MPSA92, Q7 to MPSA92, Q2 to MPSA92, Q1 to MPSA92, Q8 to MPSA92, Q3 to MPSA92
Connections:
- 595 SR pad 14: unconnected-(U6-Pad14) -> SerialSec
Routing:
- net 9v: track 0.00 -> 87.2 mm
- net Net-(D11-Pad2): track 0.00 -> 59.8 mm
- net Net-(D9-Pad2): track 0.00 -> 49.8 mm
- net Vtube: track 266.8 -> 306.6 mm
- net +5V: track 359.6 -> 397.0 mm
- net Net-(C4-Pad1): track 0.00 -> 31.6 mm
- net Net-(D9-Pad1): track 0.00 -> 19.6 mm
- net Net-(C8-Pad1): track 0.00 -> 16.1 mm
- net Net-(Q13-Pad2): track 0.00 -> 15.8 mm
- net Net-(Q13-Pad1): track 0.00 -> 15.8 mm
- net SerialSec: track 80.3 -> 94.9 mm
- net unconnected-(U6-Pad14): track 14.5 -> 0.00 mm
- net Net-(R32-Pad1): track 0.00 -> 14.3 mm
- net Net-(R27-Pad2): track 0.00 -> 9.26 mm
- net Net-(R33-Pad1): track 0.00 -> 5.77 mm
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Other:
- board size 234.1 x 84 mm -> 234 x 84 mm
- board text added: "+"
- board text added: "100k"
- board text added: "15k"
- board text added: "33k"
- board text added: "470k"
- board text added: "5v"
- board text added: "9v"
- board text added: "Gilder 2026"
- board text added: "Gnd"
- board text added: "MPSA42"
- board text added: "MPSA92"
- board text added: "Neg"
- board text added: "Nixie Pwr"
- board text added: "Pos"
- board text added: "WARNING: Higher Voltage"
